File: temp/temp.kicad_sch (KiCad schematic)
At the start: 0 parts

Commit message: Receiver & Emitter Test Firmware Complete
Parts:
- added C1: 10uF, temp:0805-NO, symbol temp-eagle-import:microbuilder_CAP_CERAMIC0805-NOOUTLINE
- added D1: RED, temp:CHIPLED_0603_NOOUTLINE, symbol temp-eagle-import:microbuilder_LED0603_NOOUTLINE
- added D2: GREEN, temp:CHIPLED_0603_NOOUTLINE, symbol temp-eagle-import:microbuilder_LED0603_NOOUTLINE
- added FID2, FID3: FIDUCIAL_1MM, temp:FIDUCIAL_1MM, symbol temp-eagle-import:microbuilder_FIDUCIAL_1MM
- added JP1: 0.1" Header, temp:1X03_OVAL, symbol temp-eagle-import:microbuilder_HEADER-1X3
- added JP3: HEADER-1X570MIL, temp:1X05_ROUND_70, symbol temp-eagle-import:microbuilder_HEADER-1X570MIL
- added O1: IRM-H6XXT, temp:IRM-H6XXT, symbol temp-eagle-import:adafruit_sensor_GENERIC_IR_RECV_IRM-H6XXT
- added O2: IRM-V5, temp:IRM-V5, symbol temp-eagle-import:adafruit_sensor_GENERIC_IR_RECV_IRM-V5
- added R1: 10K, temp:0603-NO, symbol temp-eagle-import:microbuilder_RESISTOR_0603_NOOUT
- added R3: 33K, temp:0603-NO, symbol temp-eagle-import:microbuilder_RESISTOR_0603_NOOUT
- added R4: 100, temp:0603-NO, symbol temp-eagle-import:microbuilder_RESISTOR_0603_NOOUT
- added SJ1, SJ2: SOLDERJUMPER_CLOSED, temp:SOLDERJUMPER_CLOSEDWIRE, symbol temp-eagle-import:microbuilder_SOLDERJUMPER_CLOSED
- added SW1: SPDT Slide, temp:SPDT_SMT_SSSS811101, symbol temp-eagle-import:adafruit_electromech_SWITCH_SPDT
- added U$1, U$8: MOUNTINGHOLE2.5, temp:MOUNTINGHOLE_2.5_PLATED, symbol temp-eagle-import:adafruit_electromech_MOUNTINGHOLE2.5
- added X4: JST PH 3, temp:JSTPH3, symbol temp-eagle-import:adafruit_electromech_CON_JST_PH_3PIN
Connections:
- new net: R3.2, SJ1.1
- new net: D1.C, SJ2.1
- new net: D1.A, R1.1
- new net: D2.A, R3.1
- new net: C1.1, O1.4 (VS), O2.2 (VS), R4.2
- new net GND: C1.2, D2.C, JP1.3, JP3.5, O1.1 (GND), O1.2 (GND), O2.3 (GND), O2.MT (GND), X4.1
- new net OUTH: JP3.1, O2.1 (OUT), SW1.A (O)
- new net OUTV: JP3.2, O1.3 (OUT), SW1.C (S)
- new net SIGNAL: JP1.1, JP3.3, SJ2.2, SW1.B (P), X4.3
- new net VIN: JP1.2, JP3.4, R1.2, R4.1, SJ1.2, X4.2
