File: LaserTag.kicad_sch (KiCad schematic)
At the start: 8 parts, among them SW1 SW_SPST, SW3 SW_Push, U1 TinyS3_Symbol

Commit message: attempting speaker fix
Parts:
- removed AUX_HEADER1: (no value), symbol LaserTagSymbols:LaserTag_Aux_Header
- removed U1: TinyS3_Symbol, symbol TinyS3:TinyS3_Symbol
- added BT1, BT2: Battery, symbol Device:Battery
- added LS1: Speaker, symbol Device:Speaker
- added RX2: (no value), symbol LaserTagSymbols:LaserTag_Receiver
- added SW2, SW4: SW_SPDT, symbol Switch:SW_SPDT
- added U3, U4: ESP32-C6-DevKitC-1, PCM_Espressif:ESP32-C6-DevKitC-1, symbol Espressif:ESP32-C6-DevKitC-1
Connections:
- net Button Input: now also U3.11 (GPIO11)
- net Emitter Output: now also U3.10 (GPIO10)
- net GND: now also BT2.2 (-), LS1.2, RX2.1 (GND), U3.15 (GND)
- net Receiver Input: now also U3.9 (GPIO8/BOOT)
- net V+: now also RX2.2 (V+), SW2.2 (B), U3.14 (5V)
- new net: SW4.2 (B), U4.14 (5V)
- new net: BT1.1 (+), SW4.3 (C)
- new net: BT1.2 (-), U4.15 (GND)
- new net: BT2.1 (+), SW2.3 (C)
- new net Receiver Input 2: RX2.3 (Sig), U3.23 (GPIO18)
- new net SPEAKER_OUT: LS1.1, U3.12 (GPIO2)
- no-connect marks 23 -> 57
Other:
- note added: "PLAYER MICROCONTROLLER (x3)"
- note added: "RECEIVERS"
- note added: "SERVER MICROCONTROLLER"
- note added: "SPEAKER"
- note added: "TRIGGER"
- note removed: "AUXILIARY OUTPUT"
- note removed: "BLK"
- note removed: "DIN"
- note removed: "IO36"
- note removed: "IO6"
- note removed: "IO7"
- note removed: "IO8"
- note removed: "IO9"
- note removed: "MICROCONTROLLER"
- note removed: "RECEIVER"
- note removed: "Receiver Input"
- note removed: "SCL"
- note removed: "SDA"
- note removed: "SERVER SWITCH"
- note removed: "WSEL"
- moved on the sheet: R1, SW1, TX1
