File: Schematic/LaserTag.kicad_sch (KiCad schematic)
At the start: 14 parts, among them SW1 SW_SPST, SW2 SW_SPDT, SW3 SW_Push, SW4 SW_SPDT, U3 ESP32-C6-DevKitC-1, U4 ESP32-C6-DevKitC-1

Commit message: Added Documentation & Videos / Pictures
Other:
- note added: "Battery Module"
- note added: "EMITTER (1 Per Player)"
- note added: "Laser Tag"
- note added: "PLAYER MICROCONTROLLER (1 Per Player)"
- note added: "RECEIVER (2 Per Player)"
- note added: "SERVER MICROCONTROLLER (1 Per Game)"
- note added: "SPEAKER (1 Per Player)"
- note added: "TRIGGER (1 Per Player)"
- note added: "Tyler Roche, Alfonso Landaverde"
- note removed: "EMITTER"
- note removed: "PLAYER MICROCONTROLLER (x3)"
- note removed: "RECEIVERS"
- note removed: "SERVER MICROCONTROLLER"
- note removed: "SPEAKER"
- note removed: "TRIGGER"
- moved on the sheet: BT1, BT2, LS1, R1, R2, RX1, RX2, SW1, SW2, SW3, SW4, TX1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
